File: LCD test board/lcdTestBoard.sch (EAGLE design)
At the start: 114 parts, among them CON2 AXE534124, IC1 4069D, U1 LP2980-ADJ, U10 TPS63030DSKT, U11 AR1020, U2 ST2378E_TSSOP, U3 MCP1662, U4 TPS62260, U5 ST2378E_TSSOP, U6 LP2980-ADJ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

Commit message: improved schematic readability
Parts:
- added C35: 10u/6.3V, rcl:C-EUC1206
- added C36: 100nF, rcl:C-EUC1206
- added R51: R, rcl:R-EU_R0603
- added R52: NC, rcl:R-EU_R0603
- C18: value 4.7u -> 10u/6.3V; device rcl:C-EUC0603 -> rcl:C-EUC1206
- C19: value 10u -> 10u/6.3V; device rcl:C-EUC0603 -> rcl:C-EUC1206
Connections:
- removed net 3.3_STEP_EN: C18.1, U10.EN
- new net N$32: R51.2, R52.1, U10.FB
- net 3.3_STEP: now also C18.1, C19.1, R51.1; no longer C19.2, U10.FB
- net GND: now also C19.2, C35.2, C36.2, R52.2; no longer C19.1
- net N$37: now also X1-1.B
- net N$38: now also X1-5.B
- net N$39: now also X1-2.B
- net N$40: now also X1-3.B
- net N$41: now also X1-7.B
- net N$42: now also X1-4.B
- net N$43: now also X1-6.B
- net N$44: now also X1-8.B
- net V: now also C35.1, C36.1, U10.EN
Other:
- note removed: "3.3V STEP DOWN"
- moved on the sheet: C18, C19, IC1A, IC1B, L4, R21, R22, R23, R24, R25, R26, R27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
